Commit message: fix mapper

File: 04_MapMyWorld/src/my_robot/urdf/my_robot.xacro (robot description, xacro)
@@ -152,4 +152,11 @@
     <dynamics damping="1.0" friction="1.0"/>
   </joint>
+  <link name="camera_rgbd_frame">
+  </link>
+  <joint name="camera_optical_joint" type="fixed">
+    <origin xyz="0 0 0" rpy="-1.5707 0 -1.5707"/>
+    <parent link="camera"/>
+    <child link="camera_rgbd_frame"/>
+  </joint>
   <link name='hokuyo'>
     <pose>0 0 0 0 0 0</pose>
@@ -184,7 +191,3 @@
     <dynamics damping="1.0" friction="1.0"/>
   </joint>
- <gazebo reference="left_wheel"><material>Gazebo/Green</material></gazebo>
- <gazebo reference="right_wheel"><material>Gazebo/Green</material></gazebo>
- <gazebo reference="chassis"><material>Gazebo/Blue</material></gazebo>
- <gazebo reference="camera"><material>Gazebo/Red</material></gazebo>
 </robot>
